File: hardware/lora-pump.kicad_sch (KiCad schematic)
At the start: 0 parts

Commit message: feat(hw): esquematico das folhas MCU e radio, simbolos proprios e gerador
Other:
- added sheet MCU (mcu.kicad_sch)
- added sheet Radio E220 (radio.kicad_sch)
Changed lines of the file:
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@@
 	(generator "eeschema")
 	(generator_version "10.0")
-	(paper "A4")
+	(paper "A3")
 	(title_block
 		(title "Controle de bomba d'agua LoRa")
 		(date "2026-10-11")
-		(rev "0.0")
+		(rev "0.1")
 		(company "gilsonfiho")
-		(comment 1 "Esqueleto: sem circuito ainda (ver hardware/docs/decisoes.md)")
+		(comment 1 "Folha raiz: um bloco por subfolha")
+	)
+	(sheet
+		(at 30 40)
+		(size 70 30)
+		(exclude_from_sim no)
+		(in_bom yes)
+		(on_board yes)
+		(dnp no)
+		(fields_autoplaced yes)
+		(stroke
+			(width 0.1524)
+			(type solid)
+		)
+		(fill
+			(color 0 0 0 0)
+		)
+		(property "Sheetname" "MCU"
+			(at 30 39 0)
+			(show_name no)
+			(do_not_autoplace no)
+			(effects
+				(font
+					(size 1.27 1.27)
+				)
+				(justify left bottom)
+			)
+		)
+		(property "Sheetfile" "mcu.kicad_sch"
+			(at 30 71 0)
+			(show_name no)
+			(do_not_autoplace no)
+			(effects
+				(font
+					(size 1.27 1.27)
+				)
+				(justify left top)
+			)
+		)
+		(instances
+			(project "lora-pump"
+				(path "/7f0c2b1e-5a3d-4c8e-9b1a-2d4e6f801001"
+					(page "2")
+				)
+			)
+		)
+	)
+	(sheet
+		(at 120 40)
+		(size 70 30)
+		(exclude_from_sim no)
+		(in_bom yes)
+		(on_board yes)
+		(dnp no)
+		(fields_autoplaced yes)
+		(stroke
+			(width 0.1524)
+			(type solid)
+		)
+		(fill
+			(color 0 0 0 0)
+		)
+		(property "Sheetname" "Radio E220"
+			(at 120 39 0)
+			(show_name no)
+			(do_not_autoplace no)
+			(effects
+				(font
+					(size 1.27 1.27)
+				)
+				(justify left bottom)
+			)
+		)
+		(property "Sheetfile" "radio.kicad_sch"
+			(at 120 71 0)
+			(show_name no)
+			(do_not_autoplace no)
+			(effects
+				(font
+					(size 1.27 1.27)
+				)
+				(justify left top)
+			)
+		)
+		(instances
+			(project "lora-pump"
+				(path "/7f0c2b1e-5a3d-4c8e-9b1a-2d4e6f801001"
+					(page "3")
+				)
+			)
+		)
 	)
 	(sheet_instances
