File: hardware/emissor/io.kicad_sch (KiCad schematic)
At the start: 6 parts, among them U2 E220-900T30D, U3 E220-900T22D

Commit message: feat(hw): placas emissor e receptor com layout posicionado, 3D e STEP (hw-v0.1 em andamento)
Parts:
- removed C4: 470uF/10V, Capacitor_SMD:CP_Elec_8x10.5, symbol Device:C_Polarized
- removed C5: 100nF, Capacitor_SMD:C_0603_1608Metric, symbol Device:C
- removed R7, R8: 10k, Resistor_SMD:R_0603_1608Metric, symbol Device:R
- removed U2: E220-900T30D, lora-pump:E220-900T30D, symbol lora-pump:E220-900TxxD
- removed U3: E220-900T22D, lora-pump:E220-900T22D, symbol lora-pump:E220-900TxxD
- added C10, C9: 100nF, Capacitor_SMD:C_0603_1608Metric, symbol Device:C
- added D5, D6: PESD5V0S1BL, Diode_SMD:D_SOD-323, symbol Device:D_TVS
- added J4: BOIAS, TerminalBlock_Phoenix:TerminalBlock_Phoenix_MKDS-1,5-4-5.08_1x04_P5.08mm_Horizontal, symbol Connector:Screw_Terminal_01x04
- added R15, R16: 1k, Resistor_SMD:R_0603_1608Metric, symbol Device:R
- added R17: 10k, Resistor_SMD:R_0603_1608Metric, symbol Device:R
Connections:
- net +3V3: now also R17.1
- net GND: now also C10.2, C9.2, D5.2 (A2), D6.2 (A2), J4.2 (Pin_2), J4.4 (Pin_4)
- new net FLOAT_HIGH: C10.1, R16.2
- new net FLOAT_HIGH_IN: D6.1 (A1), J4.3 (Pin_3), R16.1
- new net FLOAT_LOW: C9.1, R15.2, R17.2
- new net FLOAT_LOW_IN: D5.1 (A1), J4.1 (Pin_1), R15.1
Other:
- note added: "Cada entrada: TVS no borne, 1 k em serie e 100 nF ao GND (filtro RC) e pull-up de 10 k para 3V3. Boia baixa -> GPIO1 (FLOAT_LOW). Boia alta -> GPIO2 (FLOAT_HIGH, pull-up R2 na folha MCU). Fechada = GND (tabela de histerese em assets/schematic.md). Sem sensor ultrassonico nesta revisao."
- note added: "ENTRADAS - 2 boias (chave seca para GND)"
- note removed: "!! O E220 TRANSMITE LOGO NO BOOT: NUNCA ENERGIZAR SEM ANTENA NO SMA DO MODULO !! A antena e o SMA-K do proprio modulo (T30D/T22D Manual, Tabela 2-2, p.5): nao ha SMA na PCB. Pinos (Tabela 3-1, p.6): 1 M0, 2 M1, 3 RXD, 4 TXD, 5 AUX, 6 VCC, 7 GND; 8-11 furos de fixacao. UART/M0/M1/AUX em 3,3 V. VCC em 5 V (>= 5,0 V para potencia plena): T30D 620 mA de pico; T22D 110 mA. Entrada maxima do RX: +10 dB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"
- note removed: "RADIO - EBYTE E220-900T30D (U2) ou E220-900T22D (U3): popular UM so"
- note removed: "TEMP: PWR_FLAG de VCC_RF sai quando a folha de alimentacao for criada."
- note removed: "TODO(hw): 470 uF e palpite; bancada usa 1000 uF"
- title: Radio: E220-900T30D / T22D -> E/S - Emissor (reservatorio)
